File: bc2014.sch (KiCad schematic (older format))
At the start: 5 parts

Commit message: update schematic: adds clock, some logic, and sort out address lines
Parts:
- added C? (x4): C, symbol Device:C
- added JP? (x3): SJP, symbol Jumper:SolderJumper_3_Bridged12
- added R? (x5): R, symbol Device:R
- added SW?: SW_Push, symbol Switch:SW_Push
- added U? (x5): 74LS32, symbol 74xx:74LS32
- added U? (x5): 74HC04, symbol 74xx:74HC04
- added Y? (x2): Crystal, symbol Device:Crystal
Connections:
- net labels added: CLK2, CS, HALT, IORQ, MREQ, OE, RD, RESET, RFSH, WE, WR
- net labels removed: S1, S2, S3
- wire segments 114 -> 217
- no-connect marks 0 -> 8

Commit message: add ch340 usb uart
Parts:
- added C? (x2): 22pF, symbol Device:C
- added C?: 100nF, symbol Device:C
- added D?: LED, symbol Device:LED
- added J?: USB_B_Micro, symbol Connector:USB_B_Micro
- added R?: 1k5, symbol Device:R
- added U?: CH340G, symbol ch34x:CH340G
- added Y?: 12MHz, symbol Device:Crystal
- U?: value 27C512PLCC -> ROM, 27C512PLCC
- U?: value CY62256 -> RAM, CY62256
- U?: value 16550-LQFP-48 -> UART, 16550-LQFP-48
Connections:
- wire segments 217 -> 247
- no-connect marks 8 -> 16
Changed lines of the file:
@@
 encoding utf-8
 Sheet 1 1
-Title ""
+Title "BC2012"
 Date ""
 Rev ""
@@
 P 6650 2300
 F 0 "U?" H 6650 3500 60  0000 C CNN
-F 1 "CY62256" H 6650 3394 60  0000 C CNN
+F 1 "RAM, CY62256" H 6650 3394 60  0000 C CNN
 F 2 "" H 6700 1450 60  0000 C CNN
 F 3 "" H 6700 1450 60  0000 C CNN
@@
 P 9350 3050
 F 0 "U?" H 9350 5018 50  0000 C CNN
-F 1 "16550-LQFP-48" H 9350 4927 50  0000 C CNN
+F 1 "UART, 16550-LQFP-48" H 9350 4927 50  0000 C CNN
 F 2 "Housings_QFP:LQFP-48_7x7mm_Pitch0.5mm" H 9350 3050 50  0001 C CIN
 F 3 "http://www.ti.com/lit/ds/symlink/pc16550d.pdf" H 9350 4836 50  0000 C CNN
@@
 Wire Wire Line
 	2400 2250 1600 2250
-Wire Wire Line
-	1600 2250 1600 1650
 Connection ~ 1600 1350
 $Comp
@@
 P 6700 4900
 F 0 "U?" H 6700 6178 50  0000 C CNN
-F 1 "27C512PLCC" H 6700 6087 50  0000 C CNN
+F 1 "ROM, 27C512PLCC" H 6700 6087 50  0000 C CNN
 F 2 "Package_LCC:PLCC-32_11.4x14.0mm_P1.27mm" H 6700 4900 50  0001 C CNN
 F 3 "http://ww1.microchip.com/downloads/en/DeviceDoc/doc0015.pdf" H 6700 4900 50  0001 C CNN
@@
 	1600 1350 3100 1350
 Wire Wire Line
-	1600 1650 1950 1650
-Connection ~ 1600 1650
-Wire Wire Line
-	1600 1650 1600 1350
-Wire Wire Line
 	2250 1650 2300 1650
 Wire Wire Line
@@
 	9350 4800 9350 4900
 NoConn ~ 8350 4350
+$Comp
+L Connector:USB_B_Micro J?
+U 1 1 5C203068
+P 10900 5050
+F 0 "J?" H 10671 5041 50  0000 R CNN
+F 1 "USB_B_Micro" H 10671 4950 50  0000 R CNN
+F 2 "" H 11050 5000 50  0001 C CNN
+F 3 "~" H 11050 5000 50  0001 C CNN
+	1    10900 5050
+	-1   0    0    -1
+$EndComp
+Wire Wire Line
+	11150 5450 11150 4700
+Wire Wire Line
+	11150 4700 9500 4700
+Wire Wire Line
+	9500 4700 9500 4800
+Wire Wire Line
+	9500 4800 9350 4800
+$Comp
+L ch34x:CH340G U?
+U 1 1 5C247944
+P 10150 5900
+F 0 "U?" H 10150 6497 60  0000 C CNN
+F 1 "CH340G" H 10150 6391 60  0000 C CNN
+F 2 "" H 10250 5700 60  0000 C CNN
+F 3 "" H 10250 5700 60  0000 C CNN
+	1    10150 5900
+	1    0    0    -1
+$EndComp
+NoConn ~ 10600 5650
+NoConn ~ 10600 5750
+NoConn ~ 10600 5850
+NoConn ~ 10600 5950
+NoConn ~ 10600 6050
+NoConn ~ 10600 6150
+NoConn ~ 10600 6250
+NoConn ~ 9700 5850
+$Comp
+L Device:Crystal Y?
+U 1 1 5C2D3E3D
+P 9500 6300
+F 0 "Y?" V 9454 6169 50  0000 R CNN
+F 1 "12MHz" V 9545 6169 50  0000 R CNN
+F 2 "" H 9500 6300 50  0001 C CNN
+F 3 "~" H 9500 6300 50  0001 C CNN
+	1    9500 6300
+	0    -1   1    0
+$EndComp
+Wire Wire Line
+	9500 6150 9700 6150
+Wire Wire Line
+	9500 6450 9700 6450
+Wire Wire Line
+	9700 6450 9700 6250
+$Comp
+L Device:C C?
+U 1 1 5C31A8BB
+P 9250 6450
+F 0 "C?" V 8998 6450 50  0000 C CNN
+F 1 "22pF" V 9089 6450 50  0000 C CNN
+F 2 "" H 9288 6300 50  0001 C CNN
+F 3 "~" H 9250 6450 50  0001 C CNN
+	1    9250 6450
+	0    1    1    0
+$EndComp
+$Comp
+L Device:C C?
+U 1 1 5C31AA22
+P 9250 6150
+F 0 "C?" V 8998 6150 50  0000 C CNN
+F 1 "22pF" V 9089 6150 50  0000 C CNN
+F 2 "" H 9288 6000 50  0001 C CNN
+F 3 "~" H 9250 6150 50  0001 C CNN
+	1    9250 6150
+	0    1    1    0
+$EndComp
+Wire Wire Line
+	9400 6150 9500 6150
+Connection ~ 9500 6150
+Wire Wire Line
+	9500 6450 9400 6450
+Connection ~ 9500 6450
+$Comp
+L power:GND #PWR?
+U 1 1 5C33EBC8
+P 9000 6650
+F 0 "#PWR?" H 9000 6400 50  0001 C CNN
+F 1 "GND" H 9005 6477 50  0000 C CNN
+F 2 "" H 9000 6650 50  0001 C CNN
+F 3 "" H 9000 6650 50  0001 C CNN
+	1    9000 6650
+	1    0    0    -1
+$EndComp
+Text GLabel 9550 5750 0    50   Input ~ 0
+TX
+Text GLabel 9550 5650 0    50   Input ~ 0
+RX
+Wire Wire Line
+	9550 5650 9700 5650
+Wire Wire Line
+	9550 5750 9700 5750
+$Comp
+L Device:C C?
+U 1 1 5C458292
+P 10750 5700
+F 0 "C?" H 10865 5746 50  0000 L CNN
+F 1 "100nF" H 10865 5655 50  0000 L CNN
+F 2 "" H 10788 5550 50  0001 C CNN
+F 3 "~" H 10750 5700 50  0001 C CNN
+	1    10750 5700
+	1    0    0    -1
+$EndComp
+Wire Wire Line
+	10400 4850 10600 4850
+Wire Wire Line
+	10750 5850 10750 6650
+Wire Wire Line
+	10750 6650 9000 6650
+Wire Wire Line
+	9000 6650 9000 6450
+Wire Wire Line
+	9000 6450 9100 6450
+Connection ~ 9000 6650
+Wire Wire Line
+	9000 6450 9000 6150
+Wire Wire Line
+	9000 6150 9100 6150
+Connection ~ 9000 6450
+Wire Wire Line
+	9000 6150 9000 5550
+Connection ~ 9000 6150
+$Comp
+L Device:LED D?
+U 1 1 5C4DDB2C
+P 10950 5700
+F 0 "D?" V 10988 5583 50  0000 R CNN
+F 1 "LED" V 10897 5583 50  0000 R CNN
+F 2 "" H 10950 5700 50  0001 C CNN
+F 3 "~" H 10950 5700 50  0001 C CNN
+	1    10950 5700
+	0    -1   -1   0
+$EndComp
+$Comp
+L Device:R R?
+U 1 1 5C52BDBF
+P 10950 6100
+F 0 "R?" H 11020 6146 50  0000 L CNN
+F 1 "1k5" H 11020 6055 50  0000 L CNN
+F 2 "" V 10880 6100 50  0001 C CNN
+F 3 "~" H 10950 6100 50  0001 C CNN
+	1    10950 6100
+	1    0    0    -1
+$EndComp
+Wire Wire Line
+	10950 5850 10950 5950
+Wire Wire Line
+	10950 6250 10950 6650
+Wire Wire Line
+	10950 6650 10750 6650
+Connection ~ 10750 6650
+Connection ~ 11000 5450
+Wire Wire Line
+	11000 5450 11150 5450
+Wire Wire Line
+	10900 5450 11000 5450
+Wire Wire Line
+	10600 5550 10600 5450
+Wire Wire Line
+	10600 5450 10400 5450
+Wire Wire Line
+	10400 5450 10400 4850
+Wire Wire Line
+	10600 5550 10750 5550
+Connection ~ 10600 5550
+Wire Wire Line
+	10750 5550 10950 5550
+Connection ~ 10750 5550
+Wire Wire Line
+	9700 5550 9000 5550
+Wire Wire Line
+	1600 1650 1600 1350
+Wire Wire Line
+	1600 2250 1600 1650
+Connection ~ 1600 1650
+Wire Wire Line
+	1600 1650 1950 1650
 $EndSCHEMATC

Commit message: 16550 fixes
Connections:
- wire segments 247 -> 252
Changed lines of the file:
@@
 Wire Wire Line
 	9350 4750 9350 4800
-Text GLabel 10500 4450 2    50   Input ~ 0
-CLK
-Wire Wire Line
-	10350 4450 10500 4450
 Text GLabel 2200 1950 0    50   Input ~ 0
 CLK
@@
 $EndComp
 Wire Wire Line
-	10350 2150 10950 2150
-Wire Wire Line
 	10350 1950 11050 1950
 Wire Wire Line
@@
 	8200 3250 8350 3250
 NoConn ~ 8350 3550
-NoConn ~ 10350 4250
 Wire Wire Line
 	10350 2050 11050 2050
@@
 	11050 1850 11050 1950
 Connection ~ 11050 1950
-Wire Wire Line
-	10350 2450 10950 2450
-Wire Wire Line
-	10950 2450 10950 2150
-Connection ~ 10950 2150
-Wire Wire Line
-	10950 2150 11050 2150
-Wire Wire Line
-	10350 2750 10950 2750
-Wire Wire Line
-	10950 2750 10950 2450
-Connection ~ 10950 2450
 NoConn ~ 10350 2550
 NoConn ~ 10350 2650
@@
 NoConn ~ 10350 3750
 NoConn ~ 10350 3850
-Wire Wire Line
-	8350 4450 8350 4800
-Wire Wire Line
-	8350 4800 9350 4800
 Connection ~ 9350 4800
 Wire Wire Line
 	9350 4800 9350 4900
-NoConn ~ 8350 4350
 $Comp
 L Connector:USB_B_Micro J?
@@
 Wire Wire Line
 	1600 1650 1950 1650
+Wire Wire Line
+	10350 4250 10350 4450
+Wire Wire Line
+	10350 2150 11050 2150
+NoConn ~ 10350 2450
+NoConn ~ 10350 2750
+Text GLabel 8250 3850 0    50   Input ~ 0
+WR
+Text GLabel 8250 4150 0    50   Input ~ 0
+RD
+Wire Wire Line
+	8250 4150 8350 4150
+Wire Wire Line
+	8250 3850 8350 3850
+Text GLabel 8250 4350 0    50   Input ~ 0
+INT
+Wire Wire Line
+	8350 3950 8000 3950
+Wire Wire Line
+	8000 3950 8000 4050
+Wire Wire Line
+	8000 4250 8350 4250
+Wire Wire Line
+	8350 4050 8000 4050
+Connection ~ 8000 4050
+Wire Wire Line
+	8000 4050 8000 4250
+Wire Wire Line
+	8000 4250 8000 4450
+Wire Wire Line
+	8000 4800 9350 4800
+Connection ~ 8000 4250
+Wire Wire Line
+	8250 4350 8350 4350
+Wire Wire Line
+	8000 4450 8350 4450
+Connection ~ 8000 4450
+Wire Wire Line
+	8000 4450 8000 4800
 $EndSCHEMATC

Commit message: lol connect the usb
Connections:
- net labels added: D+, D-
- wire segments 252 -> 262
Changed lines of the file:
@@
 $EndComp
-Wire Wire Line
-	10400 4850 10600 4850
 Wire Wire Line
 	10750 5850 10750 6650
@@
 	10600 5550 10600 5450
 Wire Wire Line
-	10600 5450 10400 5450
-Wire Wire Line
-	10400 5450 10400 4850
-Wire Wire Line
 	10600 5550 10750 5550
 Connection ~ 10600 5550
@@
 Wire Wire Line
 	8000 4450 8000 4800
+Text GLabel 10550 5050 0    50   Input ~ 0
+D+
+Text GLabel 10550 5150 0    50   Input ~ 0
+D-
+Text GLabel 9550 5950 0    50   Input ~ 0
+D+
+Text GLabel 9550 6050 0    50   Input ~ 0
+D-
+Wire Wire Line
+	9550 6050 9700 6050
+Wire Wire Line
+	9550 5950 9700 5950
+Wire Wire Line
+	10550 5050 10600 5050
+Wire Wire Line
+	10550 5150 10600 5150
+Wire Wire Line
+	10600 4850 10350 4850
+Wire Wire Line
+	10350 4850 10350 5450
+Wire Wire Line
+	10350 5450 10600 5450
+Wire Wire Line
+	10600 5250 10600 5300
+Wire Wire Line
+	10600 5300 10650 5300
+Wire Wire Line
+	10650 5300 10650 5400
+Wire Wire Line
+	10650 5400 10800 5400
+Wire Wire Line
+	10800 5400 10800 5450
+Wire Wire Line
+	10800 5450 10900 5450
+Connection ~ 10900 5450
 $EndSCHEMATC

Commit message: rename uart to correct part (yay the pins match now)
Parts:
- U?: value UART, 16550-LQFP-48 -> UART, SC16C550B-LQFP-48
Changed lines of the file:
@@
 P 9350 3050
 F 0 "U?" H 9350 5018 50  0000 C CNN
-F 1 "UART, 16550-LQFP-48" H 9350 4927 50  0000 C CNN
+F 1 "UART, SC16C550B-LQFP-48" H 9350 4927 50  0000 C CNN
 F 2 "Housings_QFP:LQFP-48_7x7mm_Pitch0.5mm" H 9350 3050 50  0001 C CIN
-F 3 "http://www.ti.com/lit/ds/symlink/pc16550d.pdf" H 9350 4836 50  0000 C CNN
+F 3 "https://www.mouser.co.uk/datasheet/2/302/SC16C550B-1127791.pdf" H 9350 4836 50  0000 C CNN
 	1    9350 3050
 	1    0    0    -1
