File: bc2014.sch (KiCad schematic (older format))
At the start: 38 parts

Commit message: add spare inverter channel for 16c550 (needs to be low, whereas RESET bus is high normallly)
Parts:
- added U?: 74HC04, symbol 74xx:74HC04
Connections:
- wire segments 262 -> 263
Changed lines of the file:
@@
 	8000 4050 8000 4250
-Wire Wire Line
-	8000 4250 8000 4450
 Wire Wire Line
 	8000 4800 9350 4800
@@
 Wire Wire Line
 	8250 4350 8350 4350
-Wire Wire Line
-	8000 4450 8350 4450
-Connection ~ 8000 4450
-Wire Wire Line
-	8000 4450 8000 4800
 Text GLabel 10550 5050 0    50   Input ~ 0
 D+
@@
 Wire Bus Line
 	5600 1250 7800 1250
+$Comp
+L 74xx:74HC04 U?
+U 1 1 5CC1208B
+P 8000 5300
+F 0 "U?" H 8000 5617 50  0000 C CNN
+F 1 "74HC04" H 8000 5526 50  0000 C CNN
+F 2 "" H 8000 5300 50  0001 C CNN
+F 3 "http://www.nxp.com/documents/data_sheet/74HC_HCT04.pdf" H 8000 5300 50  0001 C CNN
+	1    8000 5300
+	1    0    0    -1
+$EndComp
+Wire Wire Line
+	8000 4250 8000 4800
+Wire Wire Line
+	8350 4450 8350 5300
+Wire Wire Line
+	8350 5300 8300 5300
+Text GLabel 7600 5300 0    50   Input ~ 0
+RESET
+Wire Wire Line
+	7600 5300 7700 5300
 $EndSCHEMATC

Commit message: clocks, think about the clocks
Parts:
- C? (x4): value C -> 22pF
- R? (x2): value R -> 1K
- R? (x2): value R -> 1M
- Y?: value Crystal -> 7.3728MHz
- Y?: value Crystal -> 1.8432MHz
Other:
- note added: "clk2 for 16c550 uart\n1834200/(115200*16)=1\nso divisor not set in 16c550 conf"
- note added: "system clock 7.3728 / 64\n115200 baud\nusually driving 68B50 in rc2014\ncan probably be upped to 8 if clk2 used by 16c550\n"
Changed lines of the file:
@@
 P 1400 6950
 F 0 "R?" H 1470 6996 50  0000 L CNN
-F 1 "R" H 1470 6905 50  0000 L CNN
+F 1 "1K" H 1470 6905 50  0000 L CNN
 F 2 "" V 1330 6950 50  0001 C CNN
 F 3 "~" H 1400 6950 50  0001 C CNN
@@
 P 1050 6250
 F 0 "R?" V 843 6250 50  0000 C CNN
-F 1 "R" V 934 6250 50  0000 C CNN
+F 1 "1M" V 934 6250 50  0000 C CNN
 F 2 "" V 980 6250 50  0001 C CNN
 F 3 "~" H 1050 6250 50  0001 C CNN
@@
 P 700 7400
 F 0 "C?" H 815 7446 50  0000 L CNN
-F 1 "C" H 815 7355 50  0000 L CNN
+F 1 "22pF" H 815 7355 50  0000 L CNN
 F 2 "" H 738 7250 50  0001 C CNN
 F 3 "~" H 700 7400 50  0001 C CNN
@@
 P 1400 7400
 F 0 "C?" H 1515 7446 50  0000 L CNN
-F 1 "C" H 1515 7355 50  0000 L CNN
+F 1 "22pF" H 1515 7355 50  0000 L CNN
 F 2 "" H 1438 7250 50  0001 C CNN
 F 3 "~" H 1400 7400 50  0001 C CNN
@@
 P 1050 7150
 F 0 "Y?" H 1050 7418 50  0000 C CNN
-F 1 "Crystal" H 1050 7327 50  0000 C CNN
+F 1 "7.3728MHz" H 1050 7327 50  0000 C CNN
 F 2 "" H 1050 7150 50  0001 C CNN
 F 3 "~" H 1050 7150 50  0001 C CNN
@@
 P 750 5600
 F 0 "C?" H 865 5646 50  0000 L CNN
-F 1 "C" H 865 5555 50  0000 L CNN
+F 1 "22pF" H 865 5555 50  0000 L CNN
 F 2 "" H 788 5450 50  0001 C CNN
 F 3 "~" H 750 5600 50  0001 C CNN
@@
 P 1400 5600
 F 0 "C?" H 1515 5646 50  0000 L CNN
-F 1 "C" H 1515 5555 50  0000 L CNN
+F 1 "22pF" H 1515 5555 50  0000 L CNN
 F 2 "" H 1438 5450 50  0001 C CNN
 F 3 "~" H 1400 5600 50  0001 C CNN
@@
 P 1050 5450
 F 0 "Y?" H 1050 5718 50  0000 C CNN
-F 1 "Crystal" H 1050 5627 50  0000 C CNN
+F 1 "1.8432MHz" H 1050 5627 50  0000 C CNN
 F 2 "" H 1050 5450 50  0001 C CNN
 F 3 "~" H 1050 5450 50  0001 C CNN
@@
 P 1050 4550
 F 0 "R?" V 843 4550 50  0000 C CNN
-F 1 "R" V 934 4550 50  0000 C CNN
+F 1 "1M" V 934 4550 50  0000 C CNN
 F 2 "" V 980 4550 50  0001 C CNN
 F 3 "~" H 1050 4550 50  0001 C CNN
@@
 P 1400 5200
 F 0 "R?" H 1470 5246 50  0000 L CNN
-F 1 "R" H 1470 5155 50  0000 L CNN
+F 1 "1K" H 1470 5155 50  0000 L CNN
 F 2 "" V 1330 5200 50  0001 C CNN
 F 3 "~" H 1400 5200 50  0001 C CNN
@@
 	2100 5000 2200 5000
 Text GLabel 8200 3250 0    50   Input ~ 0
-CLK
+CLK2
 Wire Wire Line
 	8200 3250 8350 3250
@@
 Wire Wire Line
 	7600 5300 7700 5300
+Text Notes 1650 7200 0    50   ~ 0
+system clock 7.3728 / 64\n115200 baud\nusually driving 68B50 in rc2014\ncan probably be upped to 8 if clk2 used by 16c550\n
+Text Notes 1650 5450 0    50   ~ 0
+clk2 for 16c550 uart\n1834200/(115200*16)=1\nso divisor not set in 16c550 conf
 $EndSCHEMATC
