File: bc2014.sch (KiCad schematic (older format))
At the start: 39 parts

Commit message: assign names, values, and footprints
Parts:
- C1, C2, C3, C4, C5, C6, C7: renamed from C?; footprint (none) -> Capacitor_SMD:C_0201_0603Metric
- D1: renamed from D?; footprint (none) -> Diode_SMD:D_0201_0603Metric
- J1: renamed from J?; footprint (none) -> Connector_USB:USB_Micro-B_Amphenol_10103594-0001LF_Horizontal
- JP1, JP2, JP3: renamed from JP?; footprint (none) -> Jumper:SolderJumper-3_P1.3mm_Bridged12_Pad1.0x1.5mm
- R1: renamed from R?; value R -> 2k2; footprint (none) -> Resistor_SMD:R_0201_0603Metric
- R2: renamed from R?; value R -> 3k3; footprint (none) -> Resistor_SMD:R_0201_0603Metric
- R3, R4, R5, R6, R7: renamed from R?; footprint (none) -> Resistor_SMD:R_0201_0603Metric
- SW1: renamed from SW?; footprint (none) -> Button_Switch_THT:SW_PUSH_6mm
- U1: renamed from U?; footprint (none) -> Package_QFP:LQFP-44_10x10mm_P0.8mm
- U2: renamed from U?; footprint (none) -> Package_SO:TSOP-I-28_11.8x8mm_P0.55mm
- U5: renamed from U?; footprint (none) -> Package_SO:SOP-16_4.4x10.4mm_P1.27mm
- U6, U7, U8: renamed from U?; footprint (none) -> Package_SO:SOIC-14_3.9x8.7mm_P1.27mm
- Y1, Y2, Y3: renamed from Y?; footprint (none) -> Crystal:Crystal_SMD_HC49-SD_HandSoldering
- gave numbers to parts that had none: 2
Connections:
- wire segments 263 -> 264
Other:
- note added: "clk2 can be omitted IF\ndivisor is set to 4 in UART/ROM\nAND system at 7.3728"
